Commit message: fix camera

File: urdf/jetank_links.xacro (robot description, xacro)
@@ -128,5 +128,5 @@
     <!-- camera -->
     <xacro:links name="CAMERA" mesh="${CAMERA_mesh}" material="${CAMERA_material}" mass="${CAMERA_mass}" link_type="${CAMERA_link_type}" dim_x="${CAMERA_dim[0]}" dim_y="${CAMERA_dim[1]}" dim_z="${CAMERA_dim[2]}"  collision_xyz="${CAMERA_collision_xyz_rpy[0]} ${CAMERA_collision_xyz_rpy[1]} ${CAMERA_collision_xyz_rpy[2]}" collision_rpy="${CAMERA_collision_xyz_rpy[3]} ${CAMERA_collision_xyz_rpy[4]} ${CAMERA_collision_xyz_rpy[5]}">
-        <origin xyz="-4.481242470433245e-09 -2.2840283131486673e-09 3.780146231591175e-09" rpy="-3.139495324799226 -3.8095938720097817e-06 0.003632669126105752" />
+        <origin xyz="-4.481242470433245e-09 -2.2840283131486673e-09 3.780146231591175e-09" rpy="-3.139495324799226 ${-3.8095938720097817e-06} 0.003632669126105752" />
         <inertial>
             <origin xyz="-0.005467113295410968 -4.792118534928669e-06 0.0028147721817248163"

File: urdf/jetank_sensors.xacro (robot description, xacro)
@@ -90,18 +90,22 @@
 	<!-- All other sensors such as Camera's, LiDAR's, IMU , etc... -->
 	<!--Dummy link -->
-	<link name="CAMERA_OPTICAL"></link>
+	<link name="DUMMY_CAMERA"/>
+	<link name="CAMERA_OPTICAL"/>
 	<!-- Joint from camera to Dummy link -->
+	<joint name="dummy_camera_joint" type="fixed">
+        <origin xyz="0 0 0" rpy="0 ${PI} 0" />
+        <parent link="CAMERA" />
+		<child link="DUMMY_CAMERA" />
+	</joint>
 	<joint name="camera_optical_joint" type="fixed">
-		<origin xyz="0 0 0" rpy="0 0 0" />
-		<parent link="CAMERA" />
+		<origin xyz="0 0 0" rpy="${-PI/2} 0 ${-PI/2}" />
+		<parent link="DUMMY_CAMERA" />
 		<child link="CAMERA_OPTICAL" />
 	</joint>
-	<gazebo reference="CAMERA">
+	<gazebo reference="DUMMY_CAMERA">
 		<sensor name="camera" type="camera">
 			<pose> 0 0 0 0 0 0 </pose>
 			<visualize>true</visualize>
 			<update_rate>10</update_rate>
-			<topic>camera/image_raw</topic>
-			<gz_fram_id>CAMERA_OPTICAL</gz_fram_id>
 			<camera>
 				<camera_info_topic>camera/camera_info</camera_info_topic>
@@ -118,4 +122,6 @@
 				</clip>
 			</camera>
+			<topic>camera/image_raw</topic>
+            <gz_frame_id>CAMERA_OPTICAL</gz_frame_id>
 		</sensor>
 	</gazebo>
