Commit message: updated gazebo drive files

File: urdf/jetank.urdf (robot description, URDF)
Before this commit: robot jetank, 22 links, 21 joints
Links:
- link ANTENNA_L: geometry collision cylinder length=0.15 radius=0.01; visual mesh filename=$(find jetank_description)/meshes/ANTENNA_L.stl scale=0.001 0.001 0.001
- link ANTENNA_R: geometry collision cylinder length=0.15 radius=0.01; visual mesh filename=$(find jetank_description)/meshes/ANTENNA_R.stl scale=0.001 0.001 0.001
- link ARM_LOWER: geometry collision cylinder length=0.06 radius=0.02; visual mesh filename=$(find jetank_description)/meshes/ARM_LOWER.stl scale=0.001 0.001 0.001
- link ARM_MIDDLE: geometry collision box size=0.115 0.005 0.05; visual mesh filename=$(find jetank_description)/meshes/ARM_MIDDLE.stl scale=0.001 0.001 0.001
- link ARM_UPPER: geometry collision box size=0.05 0.005 0.05; visual mesh filename=$(find jetank_description)/meshes/ARM_UPPER.stl scale=0.001 0.001 0.001
- link BEARING: geometry collision cylinder length=0.02 radius=0.025; visual mesh filename=$(find jetank_description)/meshes/BEARING.stl scale=0.001 0.001 0.001
- link CAMERA: geometry collision box size=0.01 0.01 0.01; visual mesh filename=$(find jetank_description)/meshes/CAMERA.stl scale=0.001 0.001 0.001
- link CAM_HOLDER: geometry collision cylinder length=0.05 radius=0.02; visual mesh filename=$(find jetank_description)/meshes/CAM_HOLDER.stl scale=0.001 0.001 0.001
- link DRIVER_WHEEL_L: geometry collision cylinder length=0.025 radius=0.025; visual mesh filename=$(find jetank_description)/meshes/DRIVER_WHEEL_L.stl scale=0.001 0.001 0.001
- link DRIVER_WHEEL_R: geometry collision cylinder length=0.025 radius=0.025; visual mesh filename=$(find jetank_description)/meshes/DRIVER_WHEEL_R.stl scale=0.001 0.001 0.001
- link FREE_WHEEL_L: geometry collision cylinder length=0.025 radius=0.025; visual mesh filename=$(find jetank_description)/meshes/FREE_WHEEL_L.stl scale=0.001 0.001 0.001
- link FREE_WHEEL_R: geometry collision cylinder length=0.025 radius=0.025; visual mesh filename=$(find jetank_description)/meshes/FREE_WHEEL_R.stl scale=0.001 0.001 0.001
- link GRIPPER_BASE: geometry collision box size=0.04 0.045 0.005; visual mesh filename=$(find jetank_description)/meshes/GRIPPER_BASE.stl scale=0.001 0.001 0.001
- link GRIPPER_L1: geometry collision mesh filename=$(find jetank_description)/meshes/GRIPPER_L1.stl scale=0.001 0.001 0.001; visual mesh filename=$(find jetank_description)/meshes/GRIPPER_L1.stl scale=0.001 0.001 0.001
- link GRIPPER_L2: geometry collision mesh filename=$(find jetank_description)/meshes/GRIPPER_L2.stl scale=0.001 0.001 0.001; visual mesh filename=$(find jetank_description)/meshes/GRIPPER_L2.stl scale=0.001 0.001 0.001
- link GRIPPER_R1: geometry collision mesh filename=$(find jetank_description)/meshes/GRIPPER_R1.stl scale=0.001 0.001 0.001; visual mesh filename=$(find jetank_description)/meshes/GRIPPER_R1.stl scale=0.001 0.001 0.001
- link GRIPPER_R2: geometry collision mesh filename=$(find jetank_description)/meshes/GRIPPER_R2.stl scale=0.001 0.001 0.001; visual mesh filename=$(find jetank_description)/meshes/GRIPPER_R2.stl scale=0.001 0.001 0.001
- link SERVO_LOWER: geometry collision box size=0.04 0.04 0.015; visual mesh filename=$(find jetank_description)/meshes/SERVO_LOWER.stl scale=0.001 0.001 0.001
- link SERVO_UPPER: geometry collision box size=0.04 0.04 0.015; visual mesh filename=$(find jetank_description)/meshes/SERVO_UPPER.stl scale=0.001 0.001 0.001
- link base_link: geometry collision box size=0.2 0.1 0.065; visual mesh filename=$(find jetank_description)/meshes/base_link.stl scale=0.001 0.001 0.001
